File: amos/main_power.kicad_sch (KiCad schematic)
At the start: 16 parts, among them CN201 19V INPUT, CN202 19V JETSON, Q201 CSD18532Q5B, U201 LM74700QDBVRQ1

Commit message: update
Parts:
- CN201, CN202: footprint easyeda2kicad:XT30-TH_XT30PW-M20.G.Y -> easyeda2kicad:CONN-TH_XT30PW-M; symbol easyeda2kicad:XT30PW-M20.G.Y -> easyeda2kicad:XT30PW-M; LCSC Part C30170175 -> C431092; MPN XT30PW-M20.G.Y -> XT30PW-M30.G.Y
- U201: value LM74700QDBVRQ1 -> LM74700QDBVTQ1; footprint easyeda2kicad:SOT-23-6_L2.9-W1.6-P0.95-LS2.8-BL -> easyeda2kicad:SOT-23-6_L2.9-W1.6-P0.95-LS2.8-TL; symbol easyeda2kicad:LM74700QDBVRQ1 -> easyeda2kicad:LM74700QDBVTQ1; LCSC Part C2941042 -> C2653623; MPN LM74700QDBVRQ1 -> LM74700QDBVTQ1
Connections:
- net +19V: now also C203.1, C204.1; no longer C203.2, C204.2
- net GND: now also C203.2, C204.2, CN201.1 (-), CN202.1 (-); no longer C203.1, C204.1, CN201.2 (-), CN202.2 (-)
- net at C202.1, F202.2: now also CN202.2 (+); no longer CN202.1 (+)
- net at F201.1: now also CN201.2 (+); no longer CN201.1 (+)
Other:
- moved on the sheet: C203, C204
Changed lines of the file:
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@@
 	)
 	(symbol
-		(lib_id "easyeda2kicad:XT30PW-M20.G.Y")
+		(lib_id "easyeda2kicad:XT30PW-M")
 		(at 205.74 77.47 90)
 		(unit 1)
@@
 			)
 		)
-		(property "Footprint" "easyeda2kicad:XT30-TH_XT30PW-M20.G.Y"
+		(property "Footprint" "easyeda2kicad:CONN-TH_XT30PW-M"
 			(at 217.17 77.47 0)
 			(hide yes)
@@
 			)
 		)
-		(property "Datasheet" "https://www.lcsc.com/datasheet/C30170175.pdf"
+		(property "Datasheet" "https://lcsc.com/product-detail/New-Arrivals_Changzhou-Amass-Elec-XT30PW-MMale-head_C431092.html"
 			(at 219.71 77.47 0)
 			(hide yes)
@@
 			)
 		)
-		(property "MPN" "XT30PW-M20.G.Y"
+		(property "MPN" "XT30PW-M30.G.Y"
 			(at 224.79 77.47 0)
 			(hide yes)
@@
 			)
 		)
-		(property "LCSC Part" "C30170175"
+		(property "LCSC Part" "C431092"
 			(at 227.33 77.47 0)
 			(hide yes)
@@
 	)
 	(symbol
-		(lib_id "easyeda2kicad:XT30PW-M20.G.Y")
+		(lib_id "easyeda2kicad:XT30PW-M")
 		(at 99.06 77.47 270)
 		(unit 1)
@@
 			)
 		)
-		(property "Footprint" "easyeda2kicad:XT30-TH_XT30PW-M20.G.Y"
+		(property "Footprint" "easyeda2kicad:CONN-TH_XT30PW-M"
 			(at 87.63 77.47 0)
 			(hide yes)
@@
 			)
 		)
-		(property "Datasheet" "https://www.lcsc.com/datasheet/C30170175.pdf"
+		(property "Datasheet" "https://lcsc.com/product-detail/New-Arrivals_Changzhou-Amass-Elec-XT30PW-MMale-head_C431092.html"
 			(at 85.09 77.47 0)
 			(hide yes)
@@
 			)
 		)
-		(property "MPN" "XT30PW-M20.G.Y"
+		(property "MPN" "XT30PW-M30.G.Y"
 			(at 80.01 77.47 0)
 			(hide yes)
@@
 			)
 		)
-		(property "LCSC Part" "C30170175"
+		(property "LCSC Part" "C431092"
 			(at 77.47 77.47 0)
 			(hide yes)
@@
 	(symbol
 		(lib_id "easyeda2kicad:RVE470UF35V167RV084")
-		(at 139.7 139.7 90)
+		(at 139.7 139.7 270)
 		(unit 1)
 		(body_style 1)
@@
 					(size 1.27 1.27)
 				)
-				(justify right)
+				(justify left)
 			)
 		)
@@
 					(size 1.27 1.27)
 				)
-				(justify right)
+				(justify left)
 			)
 		)
 		(property "Footprint" "easyeda2kicad:CAP-SMD_BD10.0-L10.3-W10.3-LS11.3-FD"
-			(at 147.32 139.7 0)
+			(at 132.08 139.7 0)
 			(hide yes)
 			(show_name no)
@@
 		)
 		(property "Datasheet" "https://www.lcsc.com/datasheet/C5155332.pdf"
-			(at 149.86 139.7 0)
+			(at 129.54 139.7 0)
 			(hide yes)
 			(show_name no)
@@
 		)
 		(property "Manufacturer" "KNSCHA(科尼盛)"
-			(at 152.4 139.7 0)
+			(at 127 139.7 0)
 			(hide yes)
 			(show_name no)
@@
 		)
 		(property "MPN" "RVE470UF35V167RV084"
-			(at 154.94 139.7 0)
+			(at 124.46 139.7 0)
 			(hide yes)
 			(show_name no)
@@
 		)
 		(property "LCSC Part" "C5155332"
-			(at 157.48 139.7 0)
+			(at 121.92 139.7 0)
 			(hide yes)
 			(show_name no)
@@
 	)
 	(symbol
-		(lib_id "easyeda2kicad:LM74700QDBVRQ1")
+		(lib_id "easyeda2kicad:LM74700QDBVTQ1")
 		(at 143.51 76.2 0)
 		(unit 1)
@@
 			)
 		)
-		(property "Value" "LM74700QDBVRQ1"
+		(property "Value" "LM74700QDBVTQ1"
 			(at 143.51 68.58 0)
 			(show_name no)
@@
 			)
 		)
-		(property "Footprint" "easyeda2kicad:SOT-23-6_L2.9-W1.6-P0.95-LS2.8-BL"
+		(property "Footprint" "easyeda2kicad:SOT-23-6_L2.9-W1.6-P0.95-LS2.8-TL"
 			(at 143.51 86.36 0)
 			(hide yes)
@@
 			)
 		)
-		(property "Datasheet" "https://www.lcsc.com/datasheet/C2941042.pdf"
+		(property "Datasheet" "https://www.lcsc.com/datasheet/C2653623.pdf"
 			(at 143.51 88.9 0)
 			(hide yes)
@@
 			)
 		)
-		(property "MPN" "LM74700QDBVRQ1"
+		(property "MPN" "LM74700QDBVTQ1"
 			(at 143.51 93.98 0)
 			(hide yes)
@@
 			)
 		)
-		(property "LCSC Part" "C2941042"
+		(property "LCSC Part" "C2653623"
 			(at 143.51 96.52 0)
 			(hide yes)
@@
 	(symbol
 		(lib_id "easyeda2kicad:RVE470UF35V167RV084")
-		(at 114.3 139.7 90)
+		(at 114.3 139.7 270)
 		(unit 1)
 		(body_style 1)
@@
 					(size 1.27 1.27)
 				)
-				(justify right)
+				(justify left)
 			)
 		)
@@
 					(size 1.27 1.27)
 				)
-				(justify right)
+				(justify left)
 			)
 		)
 		(property "Footprint" "easyeda2kicad:CAP-SMD_BD10.0-L10.3-W10.3-LS11.3-FD"
-			(at 121.92 139.7 0)
+			(at 106.68 139.7 0)
 			(hide yes)
 			(show_name no)
@@
 		)
 		(property "Datasheet" "https://www.lcsc.com/datasheet/C5155332.pdf"
-			(at 124.46 139.7 0)
+			(at 104.14 139.7 0)
 			(hide yes)
 			(show_name no)
@@
 		)
 		(property "Manufacturer" "KNSCHA(科尼盛)"
-			(at 127 139.7 0)
+			(at 101.6 139.7 0)
 			(hide yes)
 			(show_name no)
@@
 		)
 		(property "MPN" "RVE470UF35V167RV084"
-			(at 129.54 139.7 0)
+			(at 99.06 139.7 0)
 			(hide yes)
 			(show_name no)
@@
 		)
 		(property "LCSC Part" "C5155332"
-			(at 132.08 139.7 0)
-			(hide yes)
-			(show_name no)
+			(at 96.52 139.7 0)
+			(hide yes)
+			(show_name no)

Commit message: update
Connections:
- net GND: now also U201.2 (GND)
Changed lines of the file:
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@@
+	(wire
+		(pts
+			(xy 127 76.2) (xy 129.54 76.2)
+		)
+		(stroke
+			(width 0)
+			(type default)
+		)
+	)
 	(wire
 		(pts
@@
 					(unit 1)
 				)
+			)
+		)
+	)
+	(symbol
+		(lib_id "power:GND")
+		(at 127 76.2 270)
+		(unit 1)
+		(body_style 1)
+		(exclude_from_sim no)
+		(in_bom yes)
+		(on_board yes)
+		(in_pos_files yes)
+		(dnp no)
+		(fields_autoplaced yes)
+		(property "Reference" "#PWR0129"
+			(at 120.65 76.2 0)
+			(hide yes)
+			(show_name no)
+			(do_not_autoplace no)
+			(effects
+				(font
+					(size 1.27 1.27)
+				)
+			)
+		)
+		(property "Value" "GND"
+			(at 123.19 76.1999 90)
+			(show_name no)
+			(do_not_autoplace no)
+			(effects
+				(font
+					(size 1.27 1.27)
+				)
+				(justify right)
+			)
+		)
+		(property "Footprint" ""
+			(at 127 76.2 0)
+			(hide yes)
+			(show_name no)
+			(do_not_autoplace no)
+			(effects
+				(font
+					(size 1.27 1.27)
+				)
+			)
+		)
+		(property "Datasheet" ""
+			(at 127 76.2 0)
+			(hide yes)
+			(show_name no)
+			(do_not_autoplace no)
+			(effects
+				(font
+					(size 1.27 1.27)
+				)
+			)
+		)
+		(property "Description" "Power symbol creates a global label with name \"GND\" , ground"
+			(at 127 76.2 0)
+			(hide yes)
+			(show_name no)
+			(do_not_autoplace no)
+			(effects
+				(font
+					(size 1.27 1.27)
+				)
+			)
+		)
+		(pin "1"
+		)
+		(instances
+			(project "amos"
+				(path "/049ed167-7f00-4e6e-b407-0e51a9193256/56543776-b115-482b-bfe7-6ba4e5955a1e"
+					(reference "#PWR0129")
+					(unit 1)
+				)
