File: amos/buck_1v1_3v3.kicad_sch (KiCad schematic)
At the start: 16 parts, among them U601 TLV62569DBVR, U611 TLV62569DBVR

Commit message: update
Parts:
- L601, L611: footprint Inductor_SMD:L_Sunlord_SWPA4018S -> easyeda2kicad:IND-SMD_L4.0-W4.0_LQH44PN2R2MP0L; LCSC Part (none) -> C135262; MPN (none) -> SMNR4020-2.2UH; Manufacturer (none) -> SXN
Changed lines of the file:
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@@
 			)
 		)
-		(property "Footprint" "Inductor_SMD:L_Sunlord_SWPA4018S"
+		(property "Footprint" "easyeda2kicad:IND-SMD_L4.0-W4.0_LQH44PN2R2MP0L"
 			(at 77.47 107.95 0)
 			(hide yes)
@@
 		)
 		(property "Description" "Inductor"
+			(at 77.47 107.95 0)
+			(hide yes)
+			(show_name no)
+			(do_not_autoplace no)
+			(effects
+				(font
+					(size 1.27 1.27)
+				)
+			)
+		)
+		(property "LCSC Part" "C135262"
+			(at 77.47 107.95 0)
+			(hide yes)
+			(show_name no)
+			(do_not_autoplace no)
+			(effects
+				(font
+					(size 1.27 1.27)
+				)
+			)
+		)
+		(property "MPN" "SMNR4020-2.2UH"
+			(at 77.47 107.95 0)
+			(hide yes)
+			(show_name no)
+			(do_not_autoplace no)
+			(effects
+				(font
+					(size 1.27 1.27)
+				)
+			)
+		)
+		(property "Manufacturer" "SXN"
 			(at 77.47 107.95 0)
 			(hide yes)
@@
 			)
 		)
-		(property "Footprint" "Inductor_SMD:L_Sunlord_SWPA4018S"
+		(property "Footprint" "easyeda2kicad:IND-SMD_L4.0-W4.0_LQH44PN2R2MP0L"
 			(at 176.53 107.95 0)
 			(hide yes)
@@
 			(at 176.53 107.95 0)
 			(hide yes)
+			(show_name no)
+			(do_not_autoplace no)
+			(effects
+				(font
+					(size 1.27 1.27)
+				)
+			)
+		)
+		(property "LCSC Part" "C135262"
+			(at 176.53 107.95 0)
+			(hide yes)
+			(show_name no)
+			(do_not_autoplace no)
+			(effects
+				(font
+					(size 1.27 1.27)
+				)
+			)
+		)
+		(property "MPN" "SMNR4020-2.2UH"
+			(at 176.53 107.95 0)
+			(hide yes)
+			(show_name no)
+			(do_not_autoplace no)
+			(effects
+				(font
+					(size 1.27 1.27)
+				)
+			)
+		)
+		(property "Manufacturer" "SXN"
+			(at 176.53 107.95 0)
+			(hide yes)

Commit message: update
Parts:
- added C605, C606: 4.7uF, Capacitor_SMD:C_0805_2012Metric, symbol Device:C
- added C607, C608: 22uF, Capacitor_SMD:C_0805_2012Metric, symbol Device:C
- C601, C611: LCSC Part (none) -> C1679
- C602, C612: LCSC Part (none) -> C45783
Connections:
- net +1V1: now also C608.1
- net +3V3: now also C607.1
- net +5V_USB: now also C605.1, C606.1
- net GND: now also C605.2, C606.2, C607.2, C608.2
