File: amos/buck_servo_12v.kicad_sch (KiCad schematic)
At the start: 26 parts, among them Q301 CSD18532Q5B, Q302 CSD18532Q5B, U301 LM5145RGYR

Commit message: update
Parts:
- added C308: 100pF, Capacitor_SMD:C_0603_1608Metric, symbol Device:C
- added R312: 2.2, easyeda2kicad:R_0603, symbol Device:R
- C304: value 680uF -> 680pF; footprint easyeda2kicad:CAP-SMD_BD10.0-L10.3-W10.3-LS11.3-FD -> Capacitor_SMD:C_0402_1005Metric
- L301: footprint Inductor_SMD:L_Vishay_IHLP-4040 -> easyeda2kicad:IND-SMD_L13.5-W12.6; LCSC Part (none) -> C2880057; MPN (none) -> TMPA1265SP-4R7MN-D; Manufacturer (none) -> TAI-TECH
Connections:
- net GND: now also C308.2
- net at C307.2, L301.1, Q301.1 (S)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: now also R312.1
- new net: C308.1, R312.2

Commit message: update
Parts:
- added C309: 100nF 100V, symbol Device:C
- added C310, C311, C312, C313, C314: 4.7uF 100V, easyeda2kicad:CAP-SMD_BD10.0-L10.3-W10.3-LS11.3-FD, symbol easyeda2kicad:RVE470UF35V167RV084
- added C315, C316, C317, C318: 47uF 16V, easyeda2kicad:CAP-SMD_BD10.0-L10.3-W10.3-LS11.3-FD, symbol easyeda2kicad:RVE470UF35V167RV084
- added C319, C320: 22uF 16V, easyeda2kicad:CAP-SMD_BD10.0-L10.3-W10.3-LS11.3-FD, symbol easyeda2kicad:RVE470UF35V167RV084
- added C321, C322: 470uF 25V, easyeda2kicad:CAP-SMD_BD10.0-L10.3-W10.3-LS11.3-FD, symbol easyeda2kicad:RVE470UF35V167RV084
Connections:
- net +12V_SERVO: now also C315.1, C316.1, C317.1, C318.1, C319.1, C320.1, C321.1, C322.1
- net +19V: now also C309.1, C310.1, C311.1, C312.1, C313.1, C314.1
- net GND: now also C309.2, C310.2, C311.2, C312.2, C313.2, C314.2, C315.2, C316.2, C317.2, C318.2, C319.2, C320.2, C321.2, C322.2

Commit message: update
Parts:
- C309: footprint (none) -> Capacitor_SMD:C_0805_2012Metric; LCSC Part (none) -> C28233
- C310, C311, C312, C313, C314: footprint easyeda2kicad:CAP-SMD_BD10.0-L10.3-W10.3-LS11.3-FD -> Capacitor_SMD:C_1210_3225Metric; symbol easyeda2kicad:RVE470UF35V167RV084 -> Device:C; LCSC Part C5155332 -> C342614; MPN RVE470UF35V167RV084 -> (none); Manufacturer KNSCHA(科尼盛) -> (none)
- C315, C316, C317, C318: footprint easyeda2kicad:CAP-SMD_BD10.0-L10.3-W10.3-LS11.3-FD -> Capacitor_SMD:C_1210_3225Metric; symbol easyeda2kicad:RVE470UF35V167RV084 -> Device:C; LCSC Part C5155332 -> C77101; MPN RVE470UF35V167RV084 -> (none); Manufacturer KNSCHA(科尼盛) -> (none)
- C319, C320: value 22uF 16V -> 22uF 25V; footprint easyeda2kicad:CAP-SMD_BD10.0-L10.3-W10.3-LS11.3-FD -> Capacitor_SMD:C_1210_3225Metric; symbol easyeda2kicad:RVE470UF35V167RV084 -> Device:C; LCSC Part C5155332 -> C2918511; MPN RVE470UF35V167RV084 -> (none); Manufacturer KNSCHA(科尼盛) -> (none)
- C321, C322: footprint easyeda2kicad:CAP-SMD_BD10.0-L10.3-W10.3-LS11.3-FD -> easyeda2kicad:CAP-SMD_BD8.0-L8.3-W8.3-LS9.0-FD_H10.5; symbol easyeda2kicad:RVE470UF35V167RV084 -> Device:C; LCSC Part C5155332 -> C46550466; MPN RVE470UF35V167RV084 -> (none); Manufacturer KNSCHA(科尼盛) -> (none)
