File: amos/buck_servo_5v.kicad_sch (KiCad schematic)
At the start: 26 parts, among them Q401 CSD18532Q5B, Q402 CSD18532Q5B, U401 LM5145RGYR

Commit message: update
Parts:
- added C409: 100pF, Capacitor_SMD:C_0603_1608Metric, symbol Device:C
- added R413: 2.2, easyeda2kicad:R_0603, symbol Device:R
- L401: LCSC Part (none) -> C845075; MPN (none) -> IHLP4040DZER3R3M01; Manufacturer (none) -> Vishay
Connections:
- net GND: now also C409.2
- net at C407.2, L401.1, Q401.1 (S)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: now also R413.1
- new net: C409.1, R413.2

Commit message: update
Parts:
- added C408: 100nF, Capacitor_SMD:C_0402_1005Metric, symbol Device:C
- added C415, C416, C417, C418, C419: 2.2uF 100V, easyeda2kicad:CAP-SMD_BD10.0-L10.3-W10.3-LS11.3-FD, symbol easyeda2kicad:RVE470UF35V167RV084
- added C420, C421, C422, C423, C424, C425: 47uF 10V, easyeda2kicad:CAP-SMD_BD10.0-L10.3-W10.3-LS11.3-FD, symbol easyeda2kicad:RVE470UF35V167RV084
- added C426: 470uF 10V, easyeda2kicad:CAP-SMD_BD10.0-L10.3-W10.3-LS11.3-FD, symbol easyeda2kicad:RVE470UF35V167RV084
- R403: value 49.9 -> 49.9k
Connections:
- net +19V: now also C408.2, C415.1, C416.1, C417.1, C418.1, C419.1
- net +5V_SERVO: now also C420.1, C421.1, C422.1, C423.1, C424.1, C425.1, C426.1
- net GND: now also C408.1, C415.2, C416.2, C417.2, C418.2, C419.2, C420.2, C421.2, C422.2, C423.2, C424.2, C425.2, C426.2

Commit message: update
Parts:
- removed D401: SS14, Diode_SMD:D_SMA, symbol Device:D_Schottky
- C415, C416, C417, C418, C419: footprint easyeda2kicad:CAP-SMD_BD10.0-L10.3-W10.3-LS11.3-FD -> Capacitor_SMD:C_1210_3225Metric; symbol easyeda2kicad:RVE470UF35V167RV084 -> Device:C; LCSC Part C5155332 -> C76686; MPN RVE470UF35V167RV084 -> (none); Manufacturer KNSCHA(科尼盛) -> (none)
- C420, C421, C422, C423, C424, C425: footprint easyeda2kicad:CAP-SMD_BD10.0-L10.3-W10.3-LS11.3-FD -> Capacitor_SMD:C_1206_3216Metric; symbol easyeda2kicad:RVE470UF35V167RV084 -> Device:C; LCSC Part C5155332 -> C96123; MPN RVE470UF35V167RV084 -> (none); Manufacturer KNSCHA(科尼盛) -> (none)
- C426: footprint easyeda2kicad:CAP-SMD_BD10.0-L10.3-W10.3-LS11.3-FD -> easyeda2kicad:CAP-SMD_BD6.3-L6.6-W6.6-LS7.3-FD-H7.7; symbol easyeda2kicad:RVE470UF35V167RV084 -> Device:C; LCSC Part C5155332 -> C46550459; MPN RVE470UF35V167RV084 -> (none); Manufacturer KNSCHA(科尼盛) -> (none)
Connections:
- net +5V_SERVO: now also C405.1, JP401.3 (B), R408.1, U401.14 (VCC)
