File: amos/buck_usb_5v.kicad_sch (KiCad schematic)
At the start: 15 parts, among them U501 TPS54560DDAR

Commit message: update
Parts:
- L501: footprint Inductor_SMD:L_Sunlord_SWPA6028S -> easyeda2kicad:IND-SMD_L10.2-W10.2_7447798720; LCSC Part (none) -> C105681; MPN (none) -> 7447798720; Manufacturer (none) -> Würth Elektronik
Changed lines of the file:
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@@
 			)
 		)
-		(property "Footprint" "Inductor_SMD:L_Sunlord_SWPA6028S"
+		(property "Footprint" "easyeda2kicad:IND-SMD_L10.2-W10.2_7447798720"
 			(at 156.21 73.66 0)
 			(hide yes)
@@
 			(at 156.21 73.66 0)
 			(hide yes)
+			(show_name no)
+			(do_not_autoplace no)
+			(effects
+				(font
+					(size 1.27 1.27)
+				)
+			)
+		)
+		(property "LCSC Part" "C105681"
+			(at 156.21 73.66 0)
+			(hide yes)
+			(show_name no)
+			(do_not_autoplace no)
+			(effects
+				(font
+					(size 1.27 1.27)
+				)
+			)
+		)
+		(property "MPN" "7447798720"
+			(at 156.21 73.66 0)
+			(hide yes)
+			(show_name no)
+			(do_not_autoplace no)
+			(effects
+				(font
+					(size 1.27 1.27)
+				)
+			)
+		)
+		(property "Manufacturer" "Würth Elektronik"
+			(at 156.21 73.66 0)
+			(hide yes)

Commit message: update
Changed lines of the file:
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@@
+		)
+	)
+	(label "D5_V190"
+		(at 116.84 86.36 180)
+		(effects
+			(font
+				(size 1.27 1.27)
+			)
+			(justify right bottom)
+		)
+	)
+	(label "D5_V50"
+		(at 160.02 73.66 0)
+		(effects
+			(font
+				(size 1.27 1.27)
+			)
+			(justify left bottom)
 		)
 	)
@@
 					(unit 1)
 				)
+			)
+		)
+	)
+	(symbol
+		(lib_id "power:+5V_USB")
+		(at 133.35 119.38 0)
+		(unit 1)
+		(body_style 1)
+		(exclude_from_sim no)
+		(in_bom yes)
+		(on_board yes)
+		(in_pos_files yes)
+		(dnp no)
+		(fields_autoplaced yes)
+		(property "Reference" "#PWR0324"
+			(at 133.35 123.19 0)
+			(hide yes)
+			(show_name no)
+			(do_not_autoplace no)
+			(effects
+				(font
+					(size 1.27 1.27)
+				)
+			)
+		)
+		(property "Value" "+5V_USB"
+			(at 133.35 114.3 0)
+			(show_name no)
+			(do_not_autoplace no)
+			(effects
+				(font
+					(size 1.27 1.27)
+				)
+			)
+		)
+		(property "Footprint" ""
+			(at 133.35 119.38 0)
+			(hide yes)
+			(show_name no)
+			(do_not_autoplace no)
+			(effects
+				(font
+					(size 1.27 1.27)
+				)
+			)
+		)
+		(property "Datasheet" ""
+			(at 133.35 119.38 0)
+			(hide yes)
+			(show_name no)
+			(do_not_autoplace no)
+			(effects
+				(font
+					(size 1.27 1.27)
+				)
+			)
+		)
+		(property "Description" "Power symbol creates a global label with name \"+5V\""
+			(at 133.35 119.38 0)
+			(hide yes)
+			(show_name no)
+			(do_not_autoplace no)
+			(effects
+				(font
+					(size 1.27 1.27)
+				)
+			)
+		)
+		(pin "1"
+		)
+		(instances
+			(project "amos"
+				(path "/049ed167-7f00-4e6e-b407-0e51a9193256/ab1c4862-f26c-48b1-b183-8bee700199c6"
+					(reference "#PWR0324")
+					(unit 1)
+				)

Commit message: update
Parts:
- added C504, C505, C506, C507: 2.2uF 100V, Capacitor_SMD:C_1210_3225Metric, symbol Device:C
- added C508, C509, C510, C511, C512, C513: 47uF 16V, Capacitor_SMD:C_1210_3225Metric, symbol Device:C
Connections:
- net +19V: now also C504.1, C505.1, C506.1, C507.1
- net +5V_USB: now also C508.1, C509.1, C510.1, C511.1, C512.1, C513.1
- net GND: now also C504.2, C505.2, C506.2, C507.2, C508.2, C509.2, C510.2, C511.2, C512.2, C513.2
