File: amos/usb_port_a.kicad_sch (KiCad schematic)
At the start: 13 parts, among them U1301 TPS2553DBVR

Commit message: update
Parts:
- added C1306: 100nF, symbol Device:C
- added C1307: 10uF, symbol Device:C
Connections:
- net +5V_USB: now also C1306.1, C1307.1
- net GND: now also C1306.2, C1307.2
- no-connect marks 0 -> 4

Commit message: update
Parts:
- C1306: footprint (none) -> Capacitor_SMD:C_0402_1005Metric; LCSC Part (none) -> C14663
- C1307: footprint (none) -> Capacitor_SMD:C_0805_2012Metric; LCSC Part (none) -> C15850
Changed lines of the file:
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@@
 			)
 		)
-		(property "Footprint" ""
+		(property "Footprint" "Capacitor_SMD:C_0805_2012Metric"
 			(at 77.1652 165.1 0)
 			(hide yes)
@@
 		(property "Description" "Unpolarized capacitor"
 			(at 76.2 161.29 0)
+			(hide yes)
+			(show_name no)
+			(do_not_autoplace no)
+			(effects
+				(font
+					(size 1.27 1.27)
+				)
+			)
+		)
+		(property "LCSC Part" "C15850"
+			(at 0 0 0)
 			(hide yes)
 			(show_name no)
@@
 			)
 		)
-		(property "Footprint" ""
+		(property "Footprint" "Capacitor_SMD:C_0402_1005Metric"
 			(at 64.4652 165.1 0)
 			(hide yes)
@@
 			(hide yes)
 			(show_name no)
+			(do_not_autoplace no)
+			(effects
+				(font
+					(size 1.27 1.27)
+				)
+			)
+		)
+		(property "LCSC Part" "C14663"
+			(at 0 0 0)
+			(hide yes)
+			(show_name no)
