File: amos/usb_port_b.kicad_sch (KiCad schematic)
At the start: 13 parts, among them U1401 TPS2553DBVR

Commit message: update
Parts:
- added C1408: 100nF, symbol Device:C
- added C1409: 10uF, symbol Device:C
Connections:
- net +5V_USB: now also C1408.1, C1409.1
- net GND: now also C1408.2, C1409.2
- no-connect marks 0 -> 4

Commit message: update
Parts:
- C1408: footprint (none) -> Capacitor_SMD:C_0402_1005Metric; LCSC Part (none) -> C14663
- C1409: footprint (none) -> Capacitor_SMD:C_0805_2012Metric; LCSC Part (none) -> C15850
Changed lines of the file:
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@@
 			)
 		)
-		(property "Footprint" ""
+		(property "Footprint" "Capacitor_SMD:C_0805_2012Metric"
 			(at 73.3552 163.83 0)
 			(hide yes)
@@
 		(property "Description" "Unpolarized capacitor"
 			(at 72.39 160.02 0)
+			(hide yes)
+			(show_name no)
+			(do_not_autoplace no)
+			(effects
+				(font
+					(size 1.27 1.27)
+				)
+			)
+		)
+		(property "LCSC Part" "C15850"
+			(at 0 0 0)
 			(hide yes)
 			(show_name no)
@@
 			)
 		)
-		(property "Footprint" ""
+		(property "Footprint" "Capacitor_SMD:C_0402_1005Metric"
 			(at 60.6552 163.83 0)
 			(hide yes)
@@
 			(hide yes)
 			(show_name no)
+			(do_not_autoplace no)
+			(effects
+				(font
+					(size 1.27 1.27)
+				)
+			)
+		)
+		(property "LCSC Part" "C14663"
+			(at 0 0 0)
+			(hide yes)
+			(show_name no)
