File: amos/usb_upstream.kicad_sch (KiCad schematic)
At the start: 12 parts, among them U704 HD3SS3220RNHR

Commit message: update
Parts:
- added C1604: 1uF, symbol Device:C
- added C1605, C1606, C1607: 100nF, symbol Device:C
Connections:
- net +3V3: now also C1607.1
- net +5V_USB: now also C1604.1, C1605.1, C1606.1
- net GND: now also C1604.2, C1605.2, C1606.2, C1607.2

Commit message: update
Parts:
- C1604: footprint (none) -> Capacitor_SMD:C_0402_1005Metric; LCSC Part (none) -> C15849
- C1605, C1606, C1607: footprint (none) -> Capacitor_SMD:C_0402_1005Metric; LCSC Part (none) -> C14663
Changed lines of the file:
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@@
 			)
 		)
-		(property "Footprint" ""
+		(property "Footprint" "Capacitor_SMD:C_0402_1005Metric"
 			(at 51.7652 162.56 0)
 			(hide yes)
@@
 		(property "Description" "Unpolarized capacitor"
 			(at 50.8 158.75 0)
+			(hide yes)
+			(show_name no)
+			(do_not_autoplace no)
+			(effects
+				(font
+					(size 1.27 1.27)
+				)
+			)
+		)
+		(property "LCSC Part" "C15849"
+			(at 0 0 0)
 			(hide yes)
 			(show_name no)
@@
 			)
 		)
-		(property "Footprint" ""
+		(property "Footprint" "Capacitor_SMD:C_0402_1005Metric"
 			(at 64.4652 162.56 0)
 			(hide yes)
@@
 		(property "Description" "Unpolarized capacitor"
 			(at 63.5 158.75 0)
+			(hide yes)
+			(show_name no)
+			(do_not_autoplace no)
+			(effects
+				(font
+					(size 1.27 1.27)
+				)
+			)
+		)
+		(property "LCSC Part" "C14663"
+			(at 0 0 0)
 			(hide yes)
 			(show_name no)
@@
 			)
 		)
-		(property "Footprint" ""
+		(property "Footprint" "Capacitor_SMD:C_0402_1005Metric"
 			(at 83.5152 162.56 0)
 			(hide yes)
@@
 		(property "Description" "Unpolarized capacitor"
 			(at 82.55 158.75 0)
+			(hide yes)
+			(show_name no)
+			(do_not_autoplace no)
+			(effects
+				(font
+					(size 1.27 1.27)
+				)
+			)
+		)
+		(property "LCSC Part" "C14663"
+			(at 0 0 0)
 			(hide yes)
 			(show_name no)
@@
 			)
 		)
-		(property "Footprint" ""
+		(property "Footprint" "Capacitor_SMD:C_0402_1005Metric"
 			(at 39.0652 152.4 0)
 			(hide yes)
@@
 			(hide yes)
 			(show_name no)
+			(do_not_autoplace no)
+			(effects
+				(font
+					(size 1.27 1.27)
+				)
+			)
+		)
+		(property "LCSC Part" "C14663"
+			(at 0 0 0)
+			(hide yes)
+			(show_name no)
