File: amos/amos.kicad_pcb (KiCad board)
At the start: 4 copper layers, 100 x 75 mm, 322 parts, among them CN1001 B3B-EH-A, CN1101 B3B-EH-A, CN1201 B3B-EH-A, CN201 19V INPUT, CN202 19V JETSON, CN901 B3B-EH-A, Q201 CSD18532Q5B, Q301 CSD18532Q5B, Q302 CSD18532Q5B, Q401 CSD18532Q5B, Q402 CSD18532Q5B, U1001 SN74LVC2G241DCU, U1002 SP3485EN-L/TR, U1003 TPS25961DRVR, U1004 TPS16630PWPR, U1005 B4B-EH-A, U1101 SN74LVC2G241DCU, U1102 SP3485EN-L/TR, U1103 TPS25961DRVR, U1104 TPS16630PWPR, U1105 B4B-EH-A, U1201 SN74LVC2G241DCU, U1202 SP3485EN-L/TR, U1203 TPS25961DRVR, U1204 TPS16630PWPR, U1205 B4B-EH-A, U1301 TPS2553DBVR, U1401 TPS2553DBVR, U1501 TPS2553DBVR, U201 LM74700QDBVRQ1, U301 LM5145RGYR, U401 LM5145RGYR, U501 TPS54560DDAR, U601 TLV62569DBVR, U611 TLV62569DBVR, U701 TUSB8041IRGCR, U704 HD3SS3220RNHR, U801 CH344Q_C2988084, U901 SN74LVC2G241DCU, U902 SP3485EN-L/TR, U903 TPS25961DRVR, U904 TPS16630PWPR, U905 B4B-EH-A, Y701 24MHz 18pF, Y801 8MHz 20pF

Commit message: update
Parts:
- added C308: 100pF, Capacitor_SMD:C_0603_1608Metric, F.Cu at (37.0, 154.9)
- added C409: 100pF, Capacitor_SMD:C_0603_1608Metric, F.Cu at (26.5, 128.0)
- added FB701: BLM18PG221SN1D, easyeda2kicad:L0603, F.Cu at (146.2, 97.2)
- added R312: 2.2, easyeda2kicad:R_0603, F.Cu at (35.0, 154.7)
- added R413: 2.2, easyeda2kicad:R_0603, F.Cu at (26.5, 130.0)
- added REF**: MountingHole_3mm_Pad, MountingHole:MountingHole_3mm_Pad, F.Cu at (193.5, 82.0)
- added REF**: MountingHole_3mm_Pad, MountingHole:MountingHole_3mm_Pad, F.Cu at (55.0, 125.0)
- added REF**: MountingHole_3mm_Pad, MountingHole:MountingHole_3mm_Pad, F.Cu at (55.0, 55.0)
- added REF**: MountingHole_3mm_Pad, MountingHole:MountingHole_3mm_Pad, F.Cu at (195.0, 125.0)
- C304: value 680uF -> 680pF; footprint easyeda2kicad:CAP-SMD_BD10.0-L10.3-W10.3-LS11.3-FD -> Capacitor_SMD:C_0402_1005Metric
- CN201, CN202: footprint easyeda2kicad:XT30-TH_XT30PW-M20.G.Y -> easyeda2kicad:CONN-TH_XT30PW-M
- JP1001, JP1101, JP1201, JP901: footprint Jumper:SolderJumper-3_P1.3mm_Bridged12_Pad1.0x1.5mm -> Connector_PinHeader_2.54mm:PinHeader_1x02_P2.54mm_Vertical
- JP1002, JP1102, JP1202, JP902: footprint Jumper:SolderJumper-3_P1.3mm_Bridged12_Pad1.0x1.5mm -> Connector_PinHeader_2.54mm:PinHeader_1x03_P2.54mm_Vertical
- L301: footprint Inductor_SMD:L_Vishay_IHLP-4040 -> easyeda2kicad:IND-SMD_L13.5-W12.6
- L501: footprint Inductor_SMD:L_Sunlord_SWPA6028S -> easyeda2kicad:IND-SMD_L10.2-W10.2_7447798720
- L601, L611: footprint Inductor_SMD:L_Sunlord_SWPA4018S -> easyeda2kicad:IND-SMD_L4.0-W4.0_LQH44PN2R2MP0L
- R1007, R1107, R1207, R907: value 27k -> 1.02k
- U1003, U1103, U1203, U903: value TPS25961DRVR -> TPS259531DSGR; footprint easyeda2kicad:WSON-6_L2.0-W2.0-P0.65-TL-EP -> easyeda2kicad:WSON-8_L2.0-W2.0-P0.50-TL-EP
- U201: value LM74700QDBVRQ1 -> LM74700QDBVTQ1; footprint easyeda2kicad:SOT-23-6_L2.9-W1.6-P0.95-LS2.8-BL -> easyeda2kicad:SOT-23-6_L2.9-W1.6-P0.95-LS2.8-TL
- moved CN901 129.5 mm to (78.4, 166.3)
- moved TP301 124.1 mm to (13.0, 160.5)
- moved U905 122.6 mm to (79.5, 161.2)
- moved R301 117.6 mm to (26.8, 170.2), turned to 180 degrees
- moved TP501 117.2 mm to (87.5, 18.3)
- moved C304 116.5 mm to (29.8, 166.8), turned to -90 degrees
- moved R302 116.5 mm to (21.8, 168.5), turned to 180 degrees
- moved R307 116.4 mm to (29.2, 168.8)
- moved D1401 116.1 mm to (170.5, 68.4), turned to 180 degrees
- moved D502 116.1 mm to (84.5, 19.2), turned to -90 degrees
- moved L1401 114.8 mm to (170.5, 71.0)
- moved R311 113.8 mm to (13.5, 164.5)
- moved U301 113.5 mm to (27.8, 154.8)
- moved R303 113.3 mm to (25.2, 168.8)
- moved R1403 113.0 mm to (174.0, 72.0), turned to 180 degrees
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Connections:
- C203 pad 1: GND -> +19V
- C203 pad 2: +19V -> GND
- C204 pad 1: GND -> +19V
- C204 pad 2: +19V -> GND
- CN201 pad 1: Net-(CN201-+) -> GND
- CN201 pad 2: GND -> Net-(CN201-+)
- CN202 pad 1: Net-(CN202-+) -> GND
- CN202 pad 2: GND -> Net-(CN202-+)
- R1007 pad 2: Net-(U1003-ILIM) -> Net-(U1003-ILM)
- R1107 pad 2: Net-(U1103-ILIM) -> Net-(U1103-ILM)
- R1207 pad 2: Net-(U1203-ILIM) -> Net-(U1203-ILM)
- R907 pad 2: Net-(U903-ILIM) -> Net-(U903-ILM)
- U1003 pad 1: Net-(U1003-OUT) -> unconnected-(U1003-dVdt-Pad1)
- U1003 pad 2: GND -> Net-(U1003-EN/UVLO)
- U1003 pad 3: Net-(U1003-ILIM) -> +5V_SERVO
- U1003 pad 4: GND -> +5V_SERVO
- U1003 pad 5: Net-(U1003-EN/UVLO) -> Net-(U1003-OUT)
- U1003 pad 6: +5V_SERVO -> unconnected-(U1003-~{FLT}-Pad6)
- U1003 pad 7: GND -> Net-(U1003-ILM)
- U1103 pad 1: Net-(U1103-OUT) -> unconnected-(U1103-dVdt-Pad1)
- U1103 pad 2: GND -> Net-(U1103-EN/UVLO)
- U1103 pad 3: Net-(U1103-ILIM) -> +5V_SERVO
- U1103 pad 4: GND -> +5V_SERVO
- U1103 pad 5: Net-(U1103-EN/UVLO) -> Net-(U1103-OUT)
- U1103 pad 6: +5V_SERVO -> unconnected-(U1103-~{FLT}-Pad6)
- U1103 pad 7: GND -> Net-(U1103-ILM)
- U1203 pad 1: Net-(U1203-OUT) -> unconnected-(U1203-dVdt-Pad1)
- U1203 pad 2: GND -> Net-(U1203-EN/UVLO)
- U1203 pad 3: Net-(U1203-ILIM) -> +5V_SERVO
- U1203 pad 4: GND -> +5V_SERVO
- U1203 pad 5: Net-(U1203-EN/UVLO) -> Net-(U1203-OUT)
- U1203 pad 6: +5V_SERVO -> unconnected-(U1203-~{FLT}-Pad6)
- U1203 pad 7: GND -> Net-(U1203-ILM)
- U701 pad 34: Net-(U701-VDD33-Pad34) -> +3V3
- U701 pad 51: +1V1 -> Net-(FB701-Pad1)
- U701 pad 52: Net-(U701-VDD33-Pad34) -> +3V3
- U701 pad 57: +1V1 -> Net-(FB701-Pad1)
- U701 pad 63: Net-(U701-VDD33-Pad34) -> +3V3
- U903 pad 1: Net-(U903-OUT) -> unconnected-(U903-dVdt-Pad1)
- U903 pad 2: GND -> Net-(U903-EN/UVLO)
- U903 pad 3: Net-(U903-ILIM) -> +5V_SERVO
- U903 pad 4: GND -> +5V_SERVO
- U903 pad 5: Net-(U903-EN/UVLO) -> Net-(U903-OUT)
- U903 pad 6: +5V_SERVO -> unconnected-(U903-~{FLT}-Pad6)
- U903 pad 7: GND -> Net-(U903-ILM)
Routing:
- net Net-(Q201-G): track 0.00 -> 16.0 mm
- net Net-(D202-A): track 0.00 -> 2.56 mm
- net +19V: track 0.00 -> 1.76 mm, vias 0 -> 17
- net Net-(U201-VCAP): track 0.00 -> 1.48 mm
- net Net-(U201-ANODE): track 0.00 -> 0.88 mm, vias 0 -> 9
- net Net-(CN202-+): track 0.00 -> 0.85 mm, vias 0 -> 3
- net Net-(CN201-+): vias 0 -> 3
- added copper zone on B.Cu, net +19V
- added copper zone on F.Cu, net +19V
- added copper zone on F.Cu, net GND
- added copper zone on B.Cu, net Net-(CN201-+)
- added copper zone on F.Cu, net Net-(CN201-+)
- added copper zone on F.Cu, net Net-(CN202-+)
- added copper zone on B.Cu, net Net-(U201-ANODE)
- added copper zone on F.Cu, net Net-(U201-ANODE)
Other:
- board size 100 x 75 mm -> 150 x 80 mm

Commit message: update
Parts:
- added C1006: 100nF, Capacitor_SMD:C_0402_1005Metric, F.Cu at (123.1, 228.2)
- added C1007: 100nF, Capacitor_SMD:C_0402_1005Metric, F.Cu at (123.1, 230.1)
- added C1008: 100nF, Capacitor_SMD:C_0402_1005Metric, F.Cu at (123.1, 232.1)
- added C1009: 100nF, Capacitor_SMD:C_0402_1005Metric, F.Cu at (123.1, 234.1)
- added C1106: 100nF, Capacitor_SMD:C_0402_1005Metric, F.Cu at (159.6, 228.1)
- added C1107: 100nF, Capacitor_SMD:C_0402_1005Metric, F.Cu at (159.6, 230.1)
- added C1108: 100nF, Capacitor_SMD:C_0402_1005Metric, F.Cu at (159.6, 232.0)
- added C1109: 100nF, Capacitor_SMD:C_0402_1005Metric, F.Cu at (159.6, 234.0)
- added C1206: 100nF, Capacitor_SMD:C_0402_1005Metric, F.Cu at (210.6, 228.1)
- added C1207: 100nF, Capacitor_SMD:C_0402_1005Metric, F.Cu at (210.6, 230.1)
- added C1208: 100nF, Capacitor_SMD:C_0402_1005Metric, F.Cu at (210.6, 232.1)
- added C1209: 100nF, Capacitor_SMD:C_0402_1005Metric, F.Cu at (210.6, 234.0)
- added C1306: 100nF, Capacitor_SMD:C_0402_1005Metric, F.Cu at (150.8, 47.0)
- added C1307: 10uF, Capacitor_SMD:C_0805_2012Metric, F.Cu at (151.6, 44.5)
- added C1408: 100nF, Capacitor_SMD:C_0402_1005Metric, F.Cu at (169.3, 46.5)
- added C1409: 10uF, Capacitor_SMD:C_0805_2012Metric, F.Cu at (170.1, 44.0)
- added C1510: 100nF, Capacitor_SMD:C_0402_1005Metric, F.Cu at (189.8, 47.0)
- added C1511: 10uF, Capacitor_SMD:C_0805_2012Metric, F.Cu at (190.6, 44.5)
- added C1604: 1uF, Capacitor_SMD:C_0402_1005Metric, F.Cu at (128.0, 38.5)
- added C1605: 100nF, Capacitor_SMD:C_0402_1005Metric, F.Cu at (128.0, 40.5)
- added C1606: 100nF, Capacitor_SMD:C_0402_1005Metric, F.Cu at (128.0, 42.4)
- added C1607: 100nF, Capacitor_SMD:C_0402_1005Metric, F.Cu at (128.0, 44.4)
- added C309: 100nF 100V, Capacitor_SMD:C_0805_2012Metric, F.Cu at (25.1, 146.0)
- added C310: 4.7uF 100V, Capacitor_SMD:C_1210_3225Metric, F.Cu at (76.0, 95.0)
- added C311: 4.7uF 100V, Capacitor_SMD:C_1210_3225Metric, F.Cu at (69.5, 103.5)
- added C312: 4.7uF 100V, Capacitor_SMD:C_1210_3225Metric, F.Cu at (76.0, 91.5)
- added C313: 4.7uF 100V, Capacitor_SMD:C_1210_3225Metric, F.Cu at (62.5, 103.5)
- added C314: 4.7uF 100V, Capacitor_SMD:C_1210_3225Metric, F.Cu at (66.0, 103.5)
- added C315: 47uF 16V, Capacitor_SMD:C_1210_3225Metric, F.Cu at (77.5, 123.0)
- added C316: 47uF 16V, Capacitor_SMD:C_1210_3225Metric, F.Cu at (88.0, 123.0)
- added C317: 47uF 16V, Capacitor_SMD:C_1210_3225Metric, F.Cu at (70.5, 123.0)
- added C318: 47uF 16V, Capacitor_SMD:C_1210_3225Metric, F.Cu at (74.0, 123.0)
- added C319: 22uF 25V, Capacitor_SMD:C_1210_3225Metric, F.Cu at (81.0, 123.0)
- added C320: 22uF 25V, Capacitor_SMD:C_1210_3225Metric, F.Cu at (84.5, 123.0)
- added C321: 470uF 25V, easyeda2kicad:CAP-SMD_BD8.0-L8.3-W8.3-LS9.0-FD_H10.5, F.Cu at (64.5, 110.5)
- added C322: 470uF 25V, easyeda2kicad:CAP-SMD_BD8.0-L8.3-W8.3-LS9.0-FD_H10.5, F.Cu at (64.5, 119.5)
- added C408: 100nF, Capacitor_SMD:C_0402_1005Metric, F.Cu at (118.0, 150.0)
- added C415: 2.2uF 100V, Capacitor_SMD:C_1210_3225Metric, F.Cu at (78.5, 76.5)
- added C416: 2.2uF 100V, Capacitor_SMD:C_1210_3225Metric, F.Cu at (82.0, 87.5)
- added C417: 2.2uF 100V, Capacitor_SMD:C_1210_3225Metric, F.Cu at (78.5, 87.5)
- added C418: 2.2uF 100V, Capacitor_SMD:C_1210_3225Metric, F.Cu at (82.0, 76.5)
- added C419: 2.2uF 100V, Capacitor_SMD:C_1210_3225Metric, F.Cu at (75.0, 76.5)
- added C420: 47uF 10V, Capacitor_SMD:C_1206_3216Metric, F.Cu at (99.0, 83.0)
- added C421: 47uF 10V, Capacitor_SMD:C_1206_3216Metric, F.Cu at (102.0, 84.0)
- added C422: 47uF 10V, Capacitor_SMD:C_1206_3216Metric, F.Cu at (104.5, 85.0)
- added C423: 47uF 10V, Capacitor_SMD:C_1206_3216Metric, F.Cu at (105.5, 94.0)
- added C424: 47uF 10V, Capacitor_SMD:C_1206_3216Metric, F.Cu at (105.5, 91.5)
- added C425: 47uF 10V, Capacitor_SMD:C_1206_3216Metric, F.Cu at (105.5, 89.0)
- added C426: 470uF 10V, easyeda2kicad:CAP-SMD_BD6.3-L6.6-W6.6-LS7.3-FD-H7.7, F.Cu at (91.5, 102.0)
- added C504: 2.2uF 100V, Capacitor_SMD:C_1210_3225Metric, F.Cu at (92.3, 25.5)
- added C505: 2.2uF 100V, Capacitor_SMD:C_1210_3225Metric, F.Cu at (92.3, 29.8)
- added C506: 2.2uF 100V, Capacitor_SMD:C_1210_3225Metric, F.Cu at (92.3, 34.0)
- added C507: 2.2uF 100V, Capacitor_SMD:C_1210_3225Metric, F.Cu at (92.3, 38.2)
- added C508: 47uF 16V, Capacitor_SMD:C_1210_3225Metric, F.Cu at (92.3, 42.5)
- added C509: 47uF 16V, Capacitor_SMD:C_1210_3225Metric, F.Cu at (98.0, 25.5)
- added C510: 47uF 16V, Capacitor_SMD:C_1210_3225Metric, F.Cu at (98.0, 29.8)
- added C511: 47uF 16V, Capacitor_SMD:C_1210_3225Metric, F.Cu at (98.0, 34.0)
- added C512: 47uF 16V, Capacitor_SMD:C_1210_3225Metric, F.Cu at (98.0, 38.2)
- added C513: 47uF 16V, Capacitor_SMD:C_1210_3225Metric, F.Cu at (98.0, 42.5)
- added C605: 4.7uF, Capacitor_SMD:C_0805_2012Metric, F.Cu at (55.1, 31.0)
- added C606: 4.7uF, Capacitor_SMD:C_0805_2012Metric, F.Cu at (55.1, 34.0)
- added C607: 22uF, Capacitor_SMD:C_0805_2012Metric, F.Cu at (55.1, 37.0)
- added C608: 22uF, Capacitor_SMD:C_0805_2012Metric, F.Cu at (55.1, 40.0)
- added C704: 100nF, Capacitor_SMD:C_0402_1005Metric, F.Cu at (184.6, 84.7)
- added C705: 4.7uF, Capacitor_SMD:C_0805_2012Metric, F.Cu at (181.0, 85.2)
- added C706: 100nF, Capacitor_SMD:C_0402_1005Metric, F.Cu at (184.6, 86.7)
- added C707: 100nF, Capacitor_SMD:C_0402_1005Metric, F.Cu at (184.6, 88.7)
- added C708: 10uF, Capacitor_SMD:C_0805_2012Metric, F.Cu at (181.0, 88.3)
- added C709: 100nF, Capacitor_SMD:C_0402_1005Metric, F.Cu at (184.6, 90.6)
- added C710: 100nF, Capacitor_SMD:C_0402_1005Metric, F.Cu at (184.6, 92.6)
- added C711: 100nF, Capacitor_SMD:C_0402_1005Metric, F.Cu at (184.6, 94.6)
- added C712: 100nF, Capacitor_SMD:C_0402_1005Metric, F.Cu at (187.5, 84.7)
- added C713: 100nF, Capacitor_SMD:C_0402_1005Metric, F.Cu at (187.5, 86.7)
- added C714: 100nF, Capacitor_SMD:C_0402_1005Metric, F.Cu at (187.5, 88.7)
- added C715: 100nF, Capacitor_SMD:C_0402_1005Metric, F.Cu at (187.5, 90.6)
- added C716: 100nF, Capacitor_SMD:C_0402_1005Metric, F.Cu at (187.5, 92.6)
- added C717: 22uF, Capacitor_SMD:C_0805_2012Metric, F.Cu at (181.0, 91.3)
- added C718: 10uF, Capacitor_SMD:C_0805_2012Metric, F.Cu at (181.0, 94.3)
- added C804: 100nF, Capacitor_SMD:C_0402_1005Metric, F.Cu at (167.5, 106.5)
- added C805: 100nF, Capacitor_SMD:C_0402_1005Metric, F.Cu at (167.5, 108.5)
- added C806: 100nF, Capacitor_SMD:C_0402_1005Metric, F.Cu at (167.5, 110.4)
- added C807: 100nF, Capacitor_SMD:C_0402_1005Metric, F.Cu at (167.5, 112.4)
- added C808: 10uF, Capacitor_SMD:C_0805_2012Metric, F.Cu at (167.2, 115.5)
- added C906: 100nF, Capacitor_SMD:C_0402_1005Metric, F.Cu at (80.5, 228.2)
- added C907: 100nF, Capacitor_SMD:C_0402_1005Metric, F.Cu at (80.5, 230.2)
- added C908: 100nF, Capacitor_SMD:C_0402_1005Metric, F.Cu at (80.5, 232.1)
- added C909: 100nF, Capacitor_SMD:C_0402_1005Metric, F.Cu at (80.5, 234.1)
- R403: value 49.9 -> 49.9k
- moved TP401 114.1 mm to (117.0, 153.0)
- moved C307 111.6 mm to (135.5, 155.5)
- moved C401 111.6 mm to (127.0, 158.0)
- moved C402 111.6 mm to (128.0, 148.5)
- moved C403 111.6 mm to (130.5, 148.5)
- moved C404 111.6 mm to (129.0, 157.0)
- moved C405 111.6 mm to (121.5, 159.5)
- moved C406 111.6 mm to (132.5, 143.5)
- moved C407 111.6 mm to (133.0, 153.5)
- moved C409 111.6 mm to (135.5, 152.0)
- moved D401 111.6 mm to (119.5, 156.0)
- moved D402 111.6 mm to (117.6, 159.5)
- moved JP301 111.6 mm to (133.0, 158.0)
- moved JP401 111.6 mm to (128.5, 140.5)
- moved R309 111.6 mm to (133.0, 155.5)
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Connections:
- C405 pad 1: Net-(D401-K) -> +5V_SERVO
- FB701 pad 1: Net-(FB701-Pad1) -> /USB Hub/D7_V110
- JP401 pad 3: Net-(D401-K) -> +5V_SERVO
- R408 pad 1: Net-(D401-K) -> +5V_SERVO
- U201 pad 2: unconnected-(U201-GND-Pad2) -> GND
- U401 pad 14: Net-(D401-K) -> +5V_SERVO
- U701 pad 13: +1V1 -> /USB Hub/D7_V110
- U701 pad 21: +1V1 -> /USB Hub/D7_V110
- U701 pad 28: +1V1 -> /USB Hub/D7_V110
- U701 pad 31: +1V1 -> /USB Hub/D7_V110
- U701 pad 5: +1V1 -> /USB Hub/D7_V110
- U701 pad 51: Net-(FB701-Pad1) -> /USB Hub/D7_V110
- U701 pad 57: Net-(FB701-Pad1) -> /USB Hub/D7_V110
- U701 pad 8: +1V1 -> /USB Hub/D7_V110
Routing:
- net Net-(Q201-G): track 16.0 -> 2.09 mm
- net Net-(U201-ANODE): track 0.88 -> 10.1 mm, vias 9 -> 0
- net Net-(D202-A): track 2.56 -> 0.00 mm
- net Net-(U201-VCAP): track 1.48 -> 3.84 mm
- net +19V: track 1.76 -> 0.12 mm, vias 17 -> 0
- net GND: track 0.00 -> 1.35 mm, vias 0 -> 1
- net Net-(CN202-+): vias 3 -> 0
- net Net-(CN201-+): vias 3 -> 0
- added copper zone on F.Cu, net +12V_SERVO
- added copper zone on F.Cu, net +5V_SERVO
- added copper zone on F.Cu, net Net-(Q302-EP)
- added copper zone on F.Cu, net Net-(Q402-EP)
- removed copper zone on B.Cu, net +19V
- removed copper zone on B.Cu, net Net-(CN201-+)
- removed copper zone on B.Cu, net Net-(U201-ANODE)

Commit message: more update
Parts:
- removed D401: SS14, Diode_SMD:D_SMA
- moved R311 89.3 mm to (90.0, 113.5), turned to 90 degrees
- moved R306 87.8 mm to (89.0, 90.0), turned to 180 degrees
- moved C309 87.3 mm to (89.0, 86.5)
- moved D302 87.3 mm to (90.0, 110.4), turned to -90 degrees
- moved R302 86.9 mm to (87.5, 98.0), turned to -90 degrees
- moved R305 86.1 mm to (89.0, 92.0), turned to 0 degrees
- moved R307 85.9 mm to (89.0, 91.0), turned to 180 degrees
- moved R303 85.5 mm to (88.0, 96.0), turned to 180 degrees
- moved C608 85.4 mm to (134.5, 71.5)
- moved C307 84.3 mm to (79.5, 92.5), turned to 90 degrees
- moved C607 83.6 mm to (123.5, 85.0), turned to 180 degrees
- moved C304 82.8 mm to (87.5, 91.5)
- moved R405 82.1 mm to (103.5, 82.0), turned to 180 degrees
- moved D601 81.8 mm to (121.0, 88.0)
- moved C301 81.7 mm to (88.0, 95.0), turned to 0 degrees
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Routing:
- net GND: track 1.35 -> 64.2 mm
- net +19V: track 0.12 -> 52.6 mm, vias 0 -> 4
- net Net-(D301-K): track 0.00 -> 44.8 mm, vias 0 -> 3
- net +5V_USB: track 0.00 -> 36.2 mm, vias 0 -> 3
- net +12V_SERVO: track 0.00 -> 35.5 mm, vias 0 -> 2
- net Net-(Q302-EP): track 0.00 -> 35.5 mm, vias 0 -> 4
- net Net-(U704-CC2): track 0.00 -> 31.0 mm, vias 0 -> 1
- net Net-(Q402-EP): track 0.00 -> 26.6 mm, vias 0 -> 2
- net Net-(D704-D1-): track 0.00 -> 23.8 mm
- net +3V3: track 0.00 -> 22.3 mm
- net Net-(D706-D2-): track 0.00 -> 21.9 mm
- net Net-(D706-D2+): track 0.00 -> 20.7 mm, vias 0 -> 2
- net Net-(D704-D1+): track 0.00 -> 20.0 mm, vias 0 -> 2
- net +1V1: track 0.00 -> 16.5 mm
- net Net-(U704-CC1): track 0.00 -> 16.3 mm, vias 0 -> 2
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- added copper zone on F.Cu, net Net-(D501-K)
- added copper zone on F.Cu, net Net-(U611-SW)
Other:
- board size 150 x 80 mm -> 149.5 x 80 mm

Commit message: trying again with better planning
Parts:
- removed the REF** at (195.0, 55.0)
- removed the REF** at (55.0, 125.0)
- removed the REF** at (55.0, 55.0)
- removed the REF** at (195.0, 125.0)
- removed TP1001, TP1101, TP1201, TP901: SHDN, TestPoint:TestPoint_Pad_1.0x1.0mm
- added REF**: MountingHole_3.2mm_M3_DIN965_Pad_TopBottom, MountingHole:MountingHole_3.2mm_M3_DIN965_Pad_TopBottom, F.Cu at (55.0, 55.0)
- added REF**: MountingHole_3.2mm_M3_DIN965_Pad_TopBottom, MountingHole:MountingHole_3.2mm_M3_DIN965_Pad_TopBottom, F.Cu at (205.0, 125.0)
- added REF**: MountingHole_3.2mm_M3_DIN965_Pad_TopBottom, MountingHole:MountingHole_3.2mm_M3_DIN965_Pad_TopBottom, F.Cu at (55.0, 125.0)
- added REF**: MountingHole_3.2mm_M3_DIN965_Pad_TopBottom, MountingHole:MountingHole_3.2mm_M3_DIN965_Pad_TopBottom, F.Cu at (205.0, 55.0)
- moved C804 106.6 mm to (230.1, 108.0)
- moved C805 106.6 mm to (230.1, 109.9)
- moved C806 106.6 mm to (230.1, 111.9)
- moved C807 106.6 mm to (230.1, 113.9)
- moved Y701 106.1 mm to (248.1, 84.1)
- moved C808 98.6 mm to (221.7, 117.8)
- moved R801 97.5 mm to (233.0, 102.1)
- moved R802 97.5 mm to (233.0, 104.0)
- moved R803 97.5 mm to (233.0, 106.0)
- moved R804 97.5 mm to (233.0, 108.0)
- moved R805 97.5 mm to (233.0, 110.0)
- moved R806 97.5 mm to (233.0, 112.0)
- moved U801 97.5 mm to (237.0, 118.5)
- moved Y801 97.5 mm to (238.1, 103.7)
- moved U701 97.5 mm to (242.2, 76.0)
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Routing:
- net +19V: track 52.6 -> 4.11 mm, vias 4 -> 0
- net Net-(D301-K): track 44.8 -> 7.35 mm, vias 3 -> 2
- net +5V_USB: track 36.2 -> 0.00 mm, vias 3 -> 0
- net +12V_SERVO: track 35.5 -> 0.99 mm, vias 2 -> 0
- net Net-(Q302-EP): track 35.5 -> 3.86 mm, vias 4 -> 0
- net Net-(U704-CC2): track 31.0 -> 0.00 mm, vias 1 -> 0
- net GND: track 64.2 -> 38.9 mm, vias 1 -> 4
- net Net-(D704-D1-): track 23.8 -> 0.00 mm
- net Net-(Q402-EP): track 26.6 -> 3.84 mm, vias 2 -> 0
- net +3V3: track 22.3 -> 0.00 mm
- net Net-(D706-D2-): track 21.9 -> 0.00 mm
- net Net-(D706-D2+): track 20.7 -> 0.00 mm, vias 2 -> 0
- net Net-(D704-D1+): track 20.0 -> 0.00 mm, vias 2 -> 0
- net +1V1: track 16.5 -> 0.00 mm
- net Net-(U704-CC1): track 16.3 -> 0.00 mm, vias 2 -> 0
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- added copper zone on In2.Cu, net +12V_SERVO
- added copper zone on In2.Cu, net +5V_SERVO
- added copper zone on F.Cu, net Net-(C902-Pad2)
- added copper zone on F.Cu, net Net-(U903-OUT)
- removed copper zone on F.Cu, net GND
- removed copper zone on F.Cu, net Net-(D501-K)
- removed copper zone on F.Cu, net Net-(U611-SW)
Other:
- board size 149.5 x 80 mm -> 160 x 80 mm
