File: amos/servo_bus_c.kicad_sch (KiCad schematic)
At the start: 33 parts, among them CN1101 B3B-EH-A, U1101 SN74LVC2G241DCU, U1102 SP3485EN-L/TR, U1103 TPS25961DRVR, U1104 TPS16630PWPR, U1105 B4B-EH-A

Commit message: update
Parts:
- JP1101: footprint Jumper:SolderJumper-3_P1.3mm_Bridged12_Pad1.0x1.5mm -> Connector_PinHeader_2.54mm:PinHeader_1x02_P2.54mm_Vertical; symbol Jumper:SolderJumper_2_Bridged -> Jumper:Jumper_2_Bridged; LCSC Part (none) -> C492401; MPN (none) -> PZ254V-11-02P; Manufacturer (none) -> XFCN
- JP1102: footprint Jumper:SolderJumper-3_P1.3mm_Bridged12_Pad1.0x1.5mm -> Connector_PinHeader_2.54mm:PinHeader_1x03_P2.54mm_Vertical; LCSC Part (none) -> C2937625; MPN (none) -> PZ254V-11-03P; Manufacturer (none) -> XFCN
- R1107: value 27k -> 1.02k
- U1103: value TPS25961DRVR -> TPS259531DSGR; footprint easyeda2kicad:WSON-6_L2.0-W2.0-P0.65-TL-EP -> easyeda2kicad:WSON-8_L2.0-W2.0-P0.50-TL-EP; symbol easyeda2kicad:TPS25961DRVR -> easyeda2kicad:TPS259531DSGR; LCSC Part C5571272 -> C2155674; MPN TPS25961DRVR -> TPS259531DSGR
Connections:
- net +5V_SERVO: now also U1103.3 (IN), U1103.4 (IN); no longer U1103.6 (IN)
- net GND: now also U1103.8 (GND), U1103.9 (GND); no longer U1103.2 (OVLO), U1103.4 (GND), U1103.7 (GND)
- net at C1104.1, C1105.2, CN1101.2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: now also U1103.5 (OUT); no longer U1103.1 (OUT)
- net at R1107.2: now also U1103.7 (ILM); no longer U1103.3 (ILIM)
- net at R1106.1: now also U1103.2 (EN/UVLO); no longer U1103.5 (EN/UVLO)
- no-connect marks 6 -> 8
Changed lines of the file:
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@@
 	)
 	(junction
-		(at 177.8 161.29)
+		(at 129.54 153.67)
 		(diameter 0)
 		(color 0 0 0 0)
 	)
 	(junction
-		(at 129.54 153.67)
+		(at 129.54 161.29)
 		(diameter 0)
 		(color 0 0 0 0)
@@
 	)
 	(junction
+		(at 147.32 161.29)
+		(diameter 0)
+		(color 0 0 0 0)
+	)
+	(junction
 		(at 172.72 40.64)
 		(diameter 0)
@@
 	)
 	(junction
-		(at 59.69 119.38)
+		(at 175.26 153.67)
 		(diameter 0)
 		(color 0 0 0 0)
 	)
 	(junction
-		(at 186.69 45.72)
+		(at 59.69 119.38)
 		(diameter 0)
 		(color 0 0 0 0)
 	)
 	(junction
-		(at 129.54 156.21)
+		(at 186.69 45.72)
 		(diameter 0)
 		(color 0 0 0 0)
@@
 	)
 	(no_connect
+		(at 175.26 161.29)
+	)
+	(no_connect
+		(at 147.32 156.21)
+	)
+	(no_connect
 		(at 184.15 63.5)
 	)
@@
 	(wire
 		(pts
+			(xy 147.32 161.29) (xy 129.54 161.29)
+		)
+		(stroke
+			(width 0)
+			(type default)
+		)
+	)
+	(wire
+		(pts
 			(xy 184.15 76.2) (xy 186.69 76.2)
 		)
@@
 	(wire
 		(pts
+			(xy 177.8 158.75) (xy 177.8 156.21)
+		)
+		(stroke
+			(width 0)
+			(type default)
+		)
+	)
+	(wire
+		(pts
 			(xy 110.49 148.59) (xy 59.69 148.59)
 		)
@@
 	(wire
 		(pts
-			(xy 177.8 158.75) (xy 177.8 161.29)
-		)
-		(stroke
-			(width 0)
-			(type default)
-		)
-	)
-	(wire
-		(pts
 			(xy 118.11 110.49) (xy 118.11 113.03)
 		)
@@
 	(wire
 		(pts
-			(xy 180.34 161.29) (xy 177.8 161.29)
-		)
-		(stroke
-			(width 0)
-			(type default)
-		)
-	)
-	(wire
-		(pts
 			(xy 54.61 119.38) (xy 59.69 119.38)
 		)
@@
 	(wire
 		(pts
-			(xy 129.54 153.67) (xy 129.54 156.21)
-		)
-		(stroke
-			(width 0)
-			(type default)
-		)
-	)
-	(wire
-		(pts
 			(xy 105.41 135.89) (xy 113.03 135.89)
 		)
@@
 	(wire
 		(pts
-			(xy 129.54 156.21) (xy 147.32 156.21)
+			(xy 147.32 163.83) (xy 147.32 161.29)
 		)
 		(stroke
@@
 	(wire
 		(pts
-			(xy 129.54 156.21) (xy 129.54 158.75)
+			(xy 129.54 153.67) (xy 129.54 158.75)
 		)
 		(stroke
@@
 	(wire
 		(pts
-			(xy 175.26 156.21) (xy 177.8 156.21)
+			(xy 175.26 153.67) (xy 175.26 156.21)
 		)
 		(stroke
@@
 	(wire
 		(pts
-			(xy 175.26 161.29) (xy 177.8 161.29)
-		)
-		(stroke
-			(width 0)
-			(type default)
-		)
-	)
-	(wire
-		(pts
 			(xy 83.82 85.09) (xy 83.82 87.63)
 		)
@@
 	)
 	(symbol
-		(lib_id "easyeda2kicad:TPS25961DRVR")
-		(at 161.29 157.48 0)
+		(lib_id "easyeda2kicad:TPS259531DSGR")
+		(at 161.29 158.75 180)
 		(unit 1)
 		(body_style 1)
@@
 			)
 		)
-		(property "Value" "TPS25961DRVR"
+		(property "Value" "TPS259531DSGR"
 			(at 161.29 148.59 0)
 			(show_name no)
@@
 			)
 		)
-		(property "Footprint" "easyeda2kicad:WSON-6_L2.0-W2.0-P0.65-TL-EP"
+		(property "Footprint" "easyeda2kicad:WSON-8_L2.0-W2.0-P0.50-TL-EP"
 			(at 161.29 168.91 0)
 			(hide yes)
@@
 			)
 		)
-		(property "Datasheet" "https://www.lcsc.com/datasheet/C5571272.pdf"
+		(property "Datasheet" "https://www.lcsc.com/datasheet/C2155674.pdf"
 			(at 161.29 171.45 0)
 			(hide yes)
@@
 			)
 		)
-		(property "MPN" "TPS25961DRVR"
+		(property "MPN" "TPS259531DSGR"
 			(at 161.29 176.53 0)
 			(hide yes)
@@
 			)
 		)
-		(property "LCSC Part" "C5571272"
+		(property "LCSC Part" "C2155674"
 			(at 161.29 179.07 0)
 			(hide yes)
@@
 			)
 		)
-		(pin "5"
+		(pin "1"
 		)
-		(pin "4"
+		(pin "2"
 		)
 		(pin "3"
 		)
-		(pin "1"
+		(pin "4"
 		)
-		(pin "2"
+		(pin "5"
+		)
+		(pin "6"
 		)
 		(pin "7"
 		)
-		(pin "6"
+		(pin "8"
+		)
+		(pin "9"
 		)
 		(instances
@@
 			)
 		)
-		(property "Value" "27k"
+		(property "Value" "1.02k"
 			(at 140.97 164.084 90)
 			(show_name no)
@@
 	)
 	(symbol
-		(lib_id "Jumper:SolderJumper_2_Bridged")
+		(lib_id "Jumper:Jumper_2_Bridged")
 		(at 191.77 76.2 0)
 		(unit 1)
@@
 			)
 		)
-		(property "Footprint" "Jumper:SolderJumper-3_P1.3mm_Bridged12_Pad1.0x1.5mm"
+		(property "Footprint" "Connector_PinHeader_2.54mm:PinHeader_1x02_P2.54mm_Vertical"
 			(at 191.77 76.2 0)
 			(hide yes)
@@
 			)
 		)
-		(property "Description" "Solder Jumper, 2-pole, closed/bridged"
+		(property "Description" "Jumper, 2-pole, closed/bridged"
 			(at 191.77 81.28 0)
 			(hide yes)
@@
 			)
 		)
+		(property "LCSC Part" "C492401"
+			(at 191.77 82.55 0)
+			(hide yes)
+			(show_name no)
+			(do_not_autoplace no)
+			(effects
+				(font
+					(size 1.27 1.27)
+				)
+			)
+		)
+		(property "MPN" "PZ254V-11-02P"
+			(at 191.77 82.55 0)
+			(hide yes)
+			(show_name no)
+			(do_not_autoplace no)
+			(effects
+				(font
+					(size 1.27 1.27)
+				)
+			)
+		)
+		(property "Manufacturer" "XFCN"
+			(at 191.77 82.55 0)
+			(hide yes)
+			(show_name no)
+			(do_not_autoplace no)
+			(effects
+				(font
+					(size 1.27 1.27)
+				)
+			)
+		)
 		(pin "2"
 		)
@@
 	)
 	(symbol
-		(lib_id "power:GND")
-		(at 180.34 161.29 90)
-		(unit 1)
-		(body_style 1)
-		(exclude_from_sim no)
-		(in_bom yes)
-		(on_board yes)
-		(in_pos_files yes)
-		(dnp no)
-		(fields_autoplaced yes)
-		(property "Reference" "#PWR0198"
-			(at 186.69 161.29 0)
-			(hide yes)
-			(show_name no)
-			(do_not_autoplace no)
-			(effects
-				(font
-					(size 1.27 1.27)
-				)
-			)
-		)
-		(property "Value" "GND"
-			(at 184.15 161.2899 90)
-			(show_name no)
-			(do_not_autoplace no)
-			(effects
-				(font
-					(size 1.27 1.27)
-				)
-				(justify right)
-			)
-		)
-		(property "Footprint" ""
-			(at 180.34 161.29 0)
-			(hide yes)
-			(show_name no)
-			(do_not_autoplace no)
-			(effects
-				(font
-					(size 1.27 1.27)
-				)
-			)
-		)
-		(property "Datasheet" ""
-			(at 180.34 161.29 0)
-			(hide yes)
-			(show_name no)
-			(do_not_autoplace no)
-			(effects
-				(font
-					(size 1.27 1.27)
-				)
-			)
-		)
-		(property "Description" "Power symbol creates a global label with name \"GND\" , ground"
-			(at 180.34 161.29 0)
-			(hide yes)
-			(show_name no)
-			(do_not_autoplace no)
-			(effects
-				(font
-					(size 1.27 1.27)
-				)
-			)
-		)
-		(pin "1"
-		)
-		(instances
-			(project "amos"
-				(path "/049ed167-7f00-4e6e-b407-0e51a9193256/b9468b49-6dd6-4316-ba30-77c73ca17b3b"
-					(reference "#PWR0198")
-					(unit 1)
-				)
-			)
-		)
-	)
-	(symbol
 		(lib_id "easyeda2kicad:TPS16630PWPR")
 		(at 172.72 66.04 0)
@@
 			)
 		)
-		(property "Footprint" "Jumper:SolderJumper-3_P1.3mm_Bridged12_Pad1.0x1.5mm"
+		(property "Footprint" "Connector_PinHeader_2.54mm:PinHeader_1x03_P2.54mm_Vertical"
 			(at 68.58 121.92 0)
 			(hide yes)
@@
 			(hide yes)
 			(show_name no)
+			(do_not_autoplace no)
+			(effects
+				(font
+					(size 1.27 1.27)
+				)
+			)
+		)
+		(property "LCSC Part" "C2937625"
+			(at 68.58 121.92 0)
+			(hide yes)
+			(show_name no)
+			(do_not_autoplace no)
+			(effects
+				(font
+					(size 1.27 1.27)
+				)
+			)
+		)
+		(property "MPN" "PZ254V-11-03P"
+			(at 68.58 121.92 0)
+			(hide yes)
+			(show_name no)
+			(do_not_autoplace no)
+			(effects
+				(font
+					(size 1.27 1.27)
+				)
+			)
+		)
+		(property "Manufacturer" "XFCN"
+			(at 68.58 121.92 0)
+			(hide yes)
+			(show_name no)

Commit message: update
Parts:
- added C1106, C1107, C1108, C1109: 100nF, symbol Device:C
Connections:
- net +12V_SERVO: now also C1109.1
- net +3V3: now also C1106.1, C1107.1
- net +5V_SERVO: now also C1108.1
- net GND: now also C1106.2, C1107.2, C1108.2, C1109.2
Other:
- moved on the sheet: R1106

Commit message: update
Parts:
- C1106, C1107, C1108, C1109: footprint (none) -> Capacitor_SMD:C_0402_1005Metric; LCSC Part (none) -> C14663
Changed lines of the file:
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@@
 			)
 		)
-		(property "Footprint" ""
+		(property "Footprint" "Capacitor_SMD:C_0402_1005Metric"
 			(at 88.5952 179.07 0)
 			(hide yes)
@@
 			)
 		)
+		(property "LCSC Part" "C14663"
+			(at 0 0 0)
+			(hide yes)
+			(show_name no)
+			(do_not_autoplace no)
+			(effects
+				(font
+					(size 1.27 1.27)
+				)
+			)
+		)
 		(pin "1"
 		)
@@
 			)
 		)
-		(property "Footprint" ""
+		(property "Footprint" "Capacitor_SMD:C_0402_1005Metric"
 			(at 75.8952 179.07 0)
 			(hide yes)
@@
 			)
 		)
+		(property "LCSC Part" "C14663"
+			(at 0 0 0)
+			(hide yes)
+			(show_name no)
+			(do_not_autoplace no)
+			(effects
+				(font
+					(size 1.27 1.27)
+				)
+			)
+		)
 		(pin "1"
 		)
@@
 			)
 		)
-		(property "Footprint" ""
+		(property "Footprint" "Capacitor_SMD:C_0402_1005Metric"
 			(at 63.1952 179.07 0)
 			(hide yes)
@@
 			)
 		)
+		(property "LCSC Part" "C14663"
+			(at 0 0 0)
+			(hide yes)
+			(show_name no)
+			(do_not_autoplace no)
+			(effects
+				(font
+					(size 1.27 1.27)
+				)
+			)
+		)
 		(pin "1"
 		)
@@
 			)
 		)
-		(property "Footprint" ""
+		(property "Footprint" "Capacitor_SMD:C_0402_1005Metric"
 			(at 50.4952 179.07 0)
 			(hide yes)
@@
 			(hide yes)
 			(show_name no)
+			(do_not_autoplace no)
+			(effects
+				(font
+					(size 1.27 1.27)
+				)
+			)
+		)
+		(property "LCSC Part" "C14663"
+			(at 0 0 0)
+			(hide yes)
+			(show_name no)

Commit message: trying again with better planning
Parts:
- removed TP1101: SHDN, TestPoint:TestPoint_Pad_1.0x1.0mm, symbol Connector:TestPoint
Changed lines of the file:
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@@
 	)
 	(junction
-		(at 189.23 73.66)
-		(diameter 0)
-		(color 0 0 0 0)
-	)
-	(junction
 		(at 148.59 71.12)
 		(diameter 0)
@@
 	(wire
 		(pts
-			(xy 189.23 73.66) (xy 191.77 73.66)
-		)
-		(stroke
-			(width 0)
-			(type default)
-		)
-	)
-	(wire
-		(pts
 			(xy 184.15 40.64) (xy 186.69 40.64)
 		)
@@
 					(unit 1)
 				)
-			)
-		)
-	)
-	(symbol
-		(lib_id "Connector:TestPoint")
-		(at 191.77 73.66 270)
-		(unit 1)
-		(body_style 1)
-		(exclude_from_sim no)
-		(in_bom yes)
-		(on_board yes)
-		(in_pos_files yes)
-		(dnp no)
-		(fields_autoplaced yes)
-		(property "Reference" "TP1101"
-			(at 196.85 72.3899 90)
-			(show_name no)
-			(do_not_autoplace no)
-			(effects
-				(font
-					(size 1.27 1.27)
-				)
-				(justify left)
-			)
-		)
-		(property "Value" "SHDN"
-			(at 196.85 74.9299 90)
-			(show_name no)
-			(do_not_autoplace no)
-			(effects
-				(font
-					(size 1.27 1.27)
-				)
-				(justify left)
-			)
-		)
-		(property "Footprint" "TestPoint:TestPoint_Pad_1.0x1.0mm"
-			(at 191.77 78.74 0)
-			(hide yes)
-			(show_name no)
-			(do_not_autoplace no)
-			(effects
-				(font
-					(size 1.27 1.27)
-				)
-			)
-		)
-		(property "Datasheet" ""
-			(at 191.77 78.74 0)
-			(hide yes)
-			(show_name no)
-			(do_not_autoplace no)
-			(effects
-				(font
-					(size 1.27 1.27)
-				)
-			)
-		)
-		(property "Description" "test point"
-			(at 191.77 73.66 0)
-			(hide yes)
-			(show_name no)
-			(do_not_autoplace no)
-			(effects
-				(font
-					(size 1.27 1.27)
-				)
-			)
-		)
-		(pin "1"
-		)
-		(instances
-			(project "amos"
-				(path "/049ed167-7f00-4e6e-b407-0e51a9193256/b9468b49-6dd6-4316-ba30-77c73ca17b3b"
-					(reference "TP1101")
-					(unit 1)
-				)
