File: amos/servo_bus_d.kicad_sch (KiCad schematic)
At the start: 33 parts, among them CN1201 B3B-EH-A, U1201 SN74LVC2G241DCU, U1202 SP3485EN-L/TR, U1203 TPS25961DRVR, U1204 TPS16630PWPR, U1205 B4B-EH-A

Commit message: update
Parts:
- JP1201: footprint Jumper:SolderJumper-3_P1.3mm_Bridged12_Pad1.0x1.5mm -> Connector_PinHeader_2.54mm:PinHeader_1x02_P2.54mm_Vertical; symbol Jumper:SolderJumper_2_Bridged -> Jumper:Jumper_2_Bridged; LCSC Part (none) -> C492401; MPN (none) -> PZ254V-11-02P; Manufacturer (none) -> XFCN
- JP1202: footprint Jumper:SolderJumper-3_P1.3mm_Bridged12_Pad1.0x1.5mm -> Connector_PinHeader_2.54mm:PinHeader_1x03_P2.54mm_Vertical; LCSC Part (none) -> C2937625; MPN (none) -> PZ254V-11-03P; Manufacturer (none) -> XFCN
- R1207: value 27k -> 1.02k
- U1203: value TPS25961DRVR -> TPS259531DSGR; footprint easyeda2kicad:WSON-6_L2.0-W2.0-P0.65-TL-EP -> easyeda2kicad:WSON-8_L2.0-W2.0-P0.50-TL-EP; symbol easyeda2kicad:TPS25961DRVR -> easyeda2kicad:TPS259531DSGR; LCSC Part C5571272 -> C2155674; MPN TPS25961DRVR -> TPS259531DSGR
Connections:
- net +5V_SERVO: now also U1203.3 (IN), U1203.4 (IN); no longer U1203.6 (IN)
- net GND: now also U1203.8 (GND), U1203.9 (GND); no longer U1203.2 (OVLO), U1203.4 (GND), U1203.7 (GND)
- net at R1206.1: now also U1203.2 (EN/UVLO); no longer U1203.5 (EN/UVLO)
- net at C1204.1, C1205.2, CN1201.2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: now also U1203.5 (OUT); no longer U1203.1 (OUT)
- net at R1207.2: now also U1203.7 (ILM); no longer U1203.3 (ILIM)
- no-connect marks 6 -> 8
Changed lines of the file:
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@@
 	)
 	(junction
-		(at 177.8 161.29)
-		(diameter 0)
-		(color 0 0 0 0)
-	)
-	(junction
 		(at 118.11 123.19)
 		(diameter 0)
@@
 	)
 	(junction
+		(at 175.26 153.67)
+		(diameter 0)
+		(color 0 0 0 0)
+	)
+	(junction
 		(at 114.3 86.36)
 		(diameter 0)
@@
 	)
 	(junction
+		(at 129.54 161.29)
+		(diameter 0)
+		(color 0 0 0 0)
+	)
+	(junction
 		(at 59.69 119.38)
 		(diameter 0)
@@
 	)
 	(junction
+		(at 147.32 161.29)
+		(diameter 0)
+		(color 0 0 0 0)
+	)
+	(junction
 		(at 76.2 133.35)
 		(diameter 0)
@@
 	)
 	(junction
-		(at 129.54 156.21)
-		(diameter 0)
-		(color 0 0 0 0)
-	)
-	(junction
 		(at 144.78 143.51)
 		(diameter 0)
@@
 	)
 	(no_connect
+		(at 175.26 161.29)
+	)
+	(no_connect
 		(at 184.15 71.12)
 	)
 	(no_connect
+		(at 147.32 156.21)
+	)
+	(no_connect
 		(at 184.15 68.58)
 	)
@@
 	(wire
 		(pts
-			(xy 175.26 156.21) (xy 177.8 156.21)
-		)
-		(stroke
-			(width 0)
-			(type default)
-		)
-	)
-	(wire
-		(pts
 			(xy 205.74 45.72) (xy 205.74 100.33)
 		)
@@
 	(wire
 		(pts
-			(xy 82.55 135.89) (xy 82.55 123.19)
+			(xy 177.8 158.75) (xy 177.8 156.21)
 		)
 		(stroke
@@
 	(wire
 		(pts
-			(xy 144.78 158.75) (xy 147.32 158.75)
+			(xy 82.55 135.89) (xy 82.55 123.19)
 		)
 		(stroke
@@
 	(wire
 		(pts
-			(xy 161.29 55.88) (xy 158.75 55.88)
+			(xy 144.78 158.75) (xy 147.32 158.75)
 		)
 		(stroke
@@
 	(wire
 		(pts
-			(xy 104.14 97.79) (xy 106.68 97.79)
+			(xy 161.29 55.88) (xy 158.75 55.88)
 		)
 		(stroke
@@
 	(wire
 		(pts
-			(xy 213.36 118.11) (xy 215.9 118.11)
+			(xy 104.14 97.79) (xy 106.68 97.79)
 		)
 		(stroke
@@
 	(wire
 		(pts
-			(xy 158.75 55.88) (xy 158.75 58.42)
+			(xy 213.36 118.11) (xy 215.9 118.11)
 		)
 		(stroke
@@
 	(wire
 		(pts
-			(xy 82.55 140.97) (xy 85.09 140.97)
+			(xy 158.75 55.88) (xy 158.75 58.42)
 		)
 		(stroke
@@
 	(wire
 		(pts
-			(xy 175.26 161.29) (xy 177.8 161.29)
+			(xy 82.55 140.97) (xy 85.09 140.97)
 		)
 		(stroke
@@
 	(wire
 		(pts
+			(xy 175.26 153.67) (xy 175.26 156.21)
+		)
+		(stroke
+			(width 0)
+			(type default)
+		)
+	)
+	(wire
+		(pts
 			(xy 76.2 130.81) (xy 76.2 133.35)
 		)
@@
 	(wire
 		(pts
-			(xy 129.54 153.67) (xy 129.54 156.21)
+			(xy 129.54 153.67) (xy 129.54 158.75)
 		)
 		(stroke
@@
 	(wire
 		(pts
-			(xy 129.54 156.21) (xy 147.32 156.21)
-		)
-		(stroke
-			(width 0)
-			(type default)
-		)
-	)
-	(wire
-		(pts
 			(xy 189.23 73.66) (xy 191.77 73.66)
 		)
@@
 	(wire
 		(pts
-			(xy 129.54 156.21) (xy 129.54 158.75)
-		)
-		(stroke
-			(width 0)
-			(type default)
-		)
-	)
-	(wire
-		(pts
 			(xy 144.78 153.67) (xy 147.32 153.67)
 		)
@@
 	(wire
 		(pts
-			(xy 180.34 161.29) (xy 177.8 161.29)
-		)
-		(stroke
-			(width 0)
-			(type default)
-		)
-	)
-	(wire
-		(pts
 			(xy 189.23 71.12) (xy 189.23 73.66)
 		)
@@
 	(wire
 		(pts
+			(xy 147.32 161.29) (xy 129.54 161.29)
+		)
+		(stroke
+			(width 0)
+			(type default)
+		)
+	)
+	(wire
+		(pts
 			(xy 196.85 76.2) (xy 199.39 76.2)
 		)
@@
 	(wire
 		(pts
-			(xy 177.8 158.75) (xy 177.8 161.29)
+			(xy 147.32 163.83) (xy 147.32 161.29)
 		)
 		(stroke
@@
 	(symbol
 		(lib_id "power:GND")
-		(at 180.34 161.29 90)
-		(unit 1)
-		(body_style 1)
-		(exclude_from_sim no)
-		(in_bom yes)
-		(on_board yes)
-		(in_pos_files yes)
-		(dnp no)
-		(fields_autoplaced yes)
-		(property "Reference" "#PWR0221"
-			(at 186.69 161.29 0)
-			(hide yes)
-			(show_name no)
-			(do_not_autoplace no)
-			(effects
-				(font
-					(size 1.27 1.27)
-				)
-			)
-		)
-		(property "Value" "GND"
-			(at 184.15 161.2899 90)
-			(show_name no)
-			(do_not_autoplace no)
-			(effects
-				(font
-					(size 1.27 1.27)
-				)
-				(justify right)
-			)
-		)
-		(property "Footprint" ""
-			(at 180.34 161.29 0)
-			(hide yes)
-			(show_name no)
-			(do_not_autoplace no)
-			(effects
-				(font
-					(size 1.27 1.27)
-				)
-			)
-		)
-		(property "Datasheet" ""
-			(at 180.34 161.29 0)
-			(hide yes)
-			(show_name no)
-			(do_not_autoplace no)
-			(effects
-				(font
-					(size 1.27 1.27)
-				)
-			)
-		)
-		(property "Description" "Power symbol creates a global label with name \"GND\" , ground"
-			(at 180.34 161.29 0)
-			(hide yes)
-			(show_name no)
-			(do_not_autoplace no)
-			(effects
-				(font
-					(size 1.27 1.27)
-				)
-			)
-		)
-		(pin "1"
-		)
-		(instances
-			(project "amos"
-				(path "/049ed167-7f00-4e6e-b407-0e51a9193256/2098a820-ca7f-4e00-b358-f264b85b0a48"
-					(reference "#PWR0221")
-					(unit 1)
-				)
-			)
-		)
-	)
-	(symbol
-		(lib_id "power:GND")
 		(at 158.75 76.2 270)
 		(unit 1)
@@
 	)
 	(symbol
-		(lib_id "easyeda2kicad:TPS25961DRVR")
-		(at 161.29 157.48 0)
+		(lib_id "easyeda2kicad:TPS259531DSGR")
+		(at 161.29 158.75 180)
 		(unit 1)
 		(body_style 1)
@@
 			)
 		)
-		(property "Value" "TPS25961DRVR"
+		(property "Value" "TPS259531DSGR"
 			(at 161.29 148.59 0)
 			(show_name no)
@@
 			)
 		)
-		(property "Footprint" "easyeda2kicad:WSON-6_L2.0-W2.0-P0.65-TL-EP"
+		(property "Footprint" "easyeda2kicad:WSON-8_L2.0-W2.0-P0.50-TL-EP"
 			(at 161.29 168.91 0)
 			(hide yes)
@@
 			)
 		)
-		(property "Datasheet" "https://www.lcsc.com/datasheet/C5571272.pdf"
+		(property "Datasheet" "https://www.lcsc.com/datasheet/C2155674.pdf"
 			(at 161.29 171.45 0)
 			(hide yes)
@@
 			)
 		)
-		(property "MPN" "TPS25961DRVR"
+		(property "MPN" "TPS259531DSGR"
 			(at 161.29 176.53 0)
 			(hide yes)
@@
 			)
 		)
-		(property "LCSC Part" "C5571272"
+		(property "LCSC Part" "C2155674"
 			(at 161.29 179.07 0)
 			(hide yes)
@@
 			)
 		)
-		(pin "5"
+		(pin "1"
 		)
-		(pin "4"
+		(pin "2"
 		)
 		(pin "3"
 		)
-		(pin "1"
+		(pin "4"
 		)
-		(pin "2"
+		(pin "5"
+		)
+		(pin "6"
 		)
 		(pin "7"
 		)
-		(pin "6"
+		(pin "8"
+		)
+		(pin "9"
 		)
 		(instances
@@
 			)
 		)
-		(property "Footprint" "Jumper:SolderJumper-3_P1.3mm_Bridged12_Pad1.0x1.5mm"
+		(property "Footprint" "Connector_PinHeader_2.54mm:PinHeader_1x03_P2.54mm_Vertical"
 			(at 68.58 121.92 0)
 			(hide yes)
@@
 			)
 		)
+		(property "LCSC Part" "C2937625"
+			(at 68.58 121.92 0)
+			(hide yes)
+			(show_name no)
+			(do_not_autoplace no)
+			(effects
+				(font
+					(size 1.27 1.27)
+				)
+			)
+		)
+		(property "MPN" "PZ254V-11-03P"
+			(at 68.58 121.92 0)
+			(hide yes)
+			(show_name no)
+			(do_not_autoplace no)
+			(effects
+				(font
+					(size 1.27 1.27)
+				)
+			)
+		)
+		(property "Manufacturer" "XFCN"
+			(at 68.58 121.92 0)
+			(hide yes)
+			(show_name no)
+			(do_not_autoplace no)
+			(effects
+				(font
+					(size 1.27 1.27)
+				)
+			)
+		)
 		(pin "1"
 		)
@@
 			)
 		)
-		(property "Value" "27k"
+		(property "Value" "1.02k"
 			(at 140.97 164.084 90)
 			(show_name no)
@@
 	)
 	(symbol
-		(lib_id "Jumper:SolderJumper_2_Bridged")
+		(lib_id "Jumper:Jumper_2_Bridged")
 		(at 191.77 76.2 0)
 		(unit 1)
@@
 			)
 		)
-		(property "Footprint" "Jumper:SolderJumper-3_P1.3mm_Bridged12_Pad1.0x1.5mm"
+		(property "Footprint" "Connector_PinHeader_2.54mm:PinHeader_1x02_P2.54mm_Vertical"
 			(at 191.77 76.2 0)
 			(hide yes)
@@
 			)
 		)
-		(property "Description" "Solder Jumper, 2-pole, closed/bridged"
+		(property "Description" "Jumper, 2-pole, closed/bridged"
 			(at 191.77 81.28 0)
 			(hide yes)
 			(show_name no)
+			(do_not_autoplace no)
+			(effects
+				(font
+					(size 1.27 1.27)
+				)
+			)
+		)
+		(property "LCSC Part" "C492401"
+			(at 191.77 82.55 0)
+			(hide yes)
+			(show_name no)
+			(do_not_autoplace no)
+			(effects
+				(font
+					(size 1.27 1.27)
+				)
+			)
+		)
+		(property "MPN" "PZ254V-11-02P"
+			(at 191.77 82.55 0)
+			(hide yes)
+			(show_name no)
+			(do_not_autoplace no)
+			(effects
+				(font
+					(size 1.27 1.27)
+				)
+			)
+		)
+		(property "Manufacturer" "XFCN"
+			(at 191.77 82.55 0)
+			(hide yes)
+			(show_name no)

Commit message: update
Parts:
- added C1206, C1207, C1208, C1209: 100nF, symbol Device:C
Connections:
- net +12V_SERVO: now also C1209.1
- net +3V3: now also C1206.1, C1207.1
- net +5V_SERVO: now also C1208.1
- net GND: now also C1206.2, C1207.2, C1208.2, C1209.2
Other:
- moved on the sheet: R1206

Commit message: update
Parts:
- C1206, C1207, C1208, C1209: footprint (none) -> Capacitor_SMD:C_0402_1005Metric; LCSC Part (none) -> C14663
Changed lines of the file:
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@@
 			)
 		)
-		(property "Footprint" ""
+		(property "Footprint" "Capacitor_SMD:C_0402_1005Metric"
 			(at 61.9252 176.53 0)
 			(hide yes)
@@
 		(property "Description" "Unpolarized capacitor"
 			(at 60.96 172.72 0)
+			(hide yes)
+			(show_name no)
+			(do_not_autoplace no)
+			(effects
+				(font
+					(size 1.27 1.27)
+				)
+			)
+		)
+		(property "LCSC Part" "C14663"
+			(at 0 0 0)
 			(hide yes)
 			(show_name no)
@@
 			)
 		)
-		(property "Footprint" ""
+		(property "Footprint" "Capacitor_SMD:C_0402_1005Metric"
 			(at 49.2252 176.53 0)
 			(hide yes)
@@
 		(property "Description" "Unpolarized capacitor"
 			(at 48.26 172.72 0)
+			(hide yes)
+			(show_name no)
+			(do_not_autoplace no)
+			(effects
+				(font
+					(size 1.27 1.27)
+				)
+			)
+		)
+		(property "LCSC Part" "C14663"
+			(at 0 0 0)
 			(hide yes)
 			(show_name no)
@@
 			)
 		)
-		(property "Footprint" ""
+		(property "Footprint" "Capacitor_SMD:C_0402_1005Metric"
 			(at 87.3252 176.53 0)
 			(hide yes)
@@
 		(property "Description" "Unpolarized capacitor"
 			(at 86.36 172.72 0)
+			(hide yes)
+			(show_name no)
+			(do_not_autoplace no)
+			(effects
+				(font
+					(size 1.27 1.27)
+				)
+			)
+		)
+		(property "LCSC Part" "C14663"
+			(at 0 0 0)
 			(hide yes)
 			(show_name no)
@@
 			)
 		)
-		(property "Footprint" ""
+		(property "Footprint" "Capacitor_SMD:C_0402_1005Metric"
 			(at 74.6252 176.53 0)
 			(hide yes)
@@
 			(hide yes)
 			(show_name no)
+			(do_not_autoplace no)
+			(effects
+				(font
+					(size 1.27 1.27)
+				)
+			)
+		)
+		(property "LCSC Part" "C14663"
+			(at 0 0 0)
+			(hide yes)
+			(show_name no)

Commit message: trying again with better planning
Parts:
- removed TP1201: SHDN, TestPoint:TestPoint_Pad_1.0x1.0mm, symbol Connector:TestPoint
Changed lines of the file:
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@@
 	)
 	(junction
-		(at 189.23 73.66)
-		(diameter 0)
-		(color 0 0 0 0)
-	)
-	(junction
 		(at 172.72 40.64)
 		(diameter 0)
@@
 	(wire
 		(pts
-			(xy 189.23 73.66) (xy 191.77 73.66)
-		)
-		(stroke
-			(width 0)
-			(type default)
-		)
-	)
-	(wire
-		(pts
 			(xy 186.69 78.74) (xy 186.69 81.28)
 		)
@@
 					(unit 1)
 				)
-			)
-		)
-	)
-	(symbol
-		(lib_id "Connector:TestPoint")
-		(at 191.77 73.66 270)
-		(unit 1)
-		(body_style 1)
-		(exclude_from_sim no)
-		(in_bom yes)
-		(on_board yes)
-		(in_pos_files yes)
-		(dnp no)
-		(fields_autoplaced yes)
-		(property "Reference" "TP1201"
-			(at 196.85 72.3899 90)
-			(show_name no)
-			(do_not_autoplace no)
-			(effects
-				(font
-					(size 1.27 1.27)
-				)
-				(justify left)
-			)
-		)
-		(property "Value" "SHDN"
-			(at 196.85 74.9299 90)
-			(show_name no)
-			(do_not_autoplace no)
-			(effects
-				(font
-					(size 1.27 1.27)
-				)
-				(justify left)
-			)
-		)
-		(property "Footprint" "TestPoint:TestPoint_Pad_1.0x1.0mm"
-			(at 191.77 78.74 0)
-			(hide yes)
-			(show_name no)
-			(do_not_autoplace no)
-			(effects
-				(font
-					(size 1.27 1.27)
-				)
-			)
-		)
-		(property "Datasheet" ""
-			(at 191.77 78.74 0)
-			(hide yes)
-			(show_name no)
-			(do_not_autoplace no)
-			(effects
-				(font
-					(size 1.27 1.27)
-				)
-			)
-		)
-		(property "Description" "test point"
-			(at 191.77 73.66 0)
-			(hide yes)
-			(show_name no)
-			(do_not_autoplace no)
-			(effects
-				(font
-					(size 1.27 1.27)
-				)
-			)
-		)
-		(pin "1"
-		)
-		(instances
-			(project "amos"
-				(path "/049ed167-7f00-4e6e-b407-0e51a9193256/2098a820-ca7f-4e00-b358-f264b85b0a48"
-					(reference "TP1201")
-					(unit 1)
-				)
